File: octelehat.sch (KiCad schematic (older format))
At the start: 33 parts, among them P1 CONN_02X20, P2 CONN_01X04, P3 CONN_01X04, P4 CONN_01X02, P5 CONN_01X04, P6 CONN_01X04, P7 CONN_01X02, U1 MAX31855KASA, U2 MAX31855KASA, U3 ADS1015

Commit message: reassign parts for open parts library
Parts:
- removed P2, P3, P5, P6: CONN_01X04, symbol CONN_01X04
- removed P7: CONN_01X02, symbol CONN_01X02
- removed R1, R2, R5, R6: 10k, symbol R
- removed R3, R7: 100k, symbol R
- removed R4, R8: 33k, symbol R
- added J1, J2, J3: GROVE-CONNECTOR-DIP-90D_4P-2.0_, SeeedOPL-Connector-2016:HW4-2.0-90D, symbol GROVE-CONNECTOR-DIP-90D_4P-2.0_
- added P3: CONN_01X02, hat-parts:Thermocouple, symbol CONN_01X02
- added R1, R2, R5, R6: SMD-RES-10K-1%-1_10W_0603_, SeeedOPL-Resistor-2016:R0603, symbol SMD-RES-10K-1%-1_10W_0603_
- added R3, R7: SMD-RES-100K-1%-1_10W_0603_, SeeedOPL-Resistor-2016:R0603, symbol SMD-RES-100K-1%-1_10W_0603_
- added R4, R8: SMD-RES-30K-1%-1_10W_0603_, SeeedOPL-Resistor-2016:R0603, symbol SMD-RES-30K-1%-1_10W_0603_
- C1, C10, C2, C3, C4, C6, C7, C8, C9: footprint (none) -> Capacitors_SMD:C_0402; MPN (none) -> CC0402KRX7R8BB104; Manufacturer (none) -> Yageo; OPL (none) -> 302010024
- C11, C5: footprint (none) -> Capacitors_SMD:C_0402; MPN (none) -> CC0402KRX7R9BB103; Manufacturer (none) -> Yageo; OPL (none) -> 302010006
- FB1, FB2, FB3, FB4: footprint (none) -> Resistors_SMD:R_0603_HandSoldering; MPN (none) -> BLM18AG121SN1D; MPN2 (none) -> BK1608HW121-T; Manufacturer (none) -> Murata; Manufacturer2 (none) -> Taiyo Yuden; OPL (none) -> 303030001
- P1: footprint Socket_Strips:Socket_Strip_Straight_2x20 -> Socket_Strips:Socket_Strip_Straight_2x20_Pitch2.54mm; MFPN (none) -> F185-1220A0BSYA1; Manufacturer (none) -> YXCON
- P2: renamed from P4; footprint (none) -> hat-parts:Thermocouple; MPN (none) -> XE-1109-001; MPN2 (none) -> 381-7564; Manufacturer (none) -> Labfacility; Manufacturer2 (none) -> RS Pro
- U1: symbol MAX31855KASA -> MAX31855KASA-RESCUE-octelehat; MPN (none) -> MAX31855KASA; Manufacturer (none) -> Maxim Integrated
- U3: renamed from U2; symbol MAX31855KASA -> MAX31855KASA-RESCUE-octelehat; MPN (none) -> MAX31855KASA; Manufacturer (none) -> Maxim Integrated
- renumbered U3 to U2
Connections:
- net +3V3: now also C6.1, P1.18 (P18), P1.2 (P2), R1.2, R2.2, R5.2, R6.2; no longer C6.2, P1.1 (P1), P1.17 (P17)
- net 5V: now also P1.1 (P1); no longer P1.2 (P2)
- net GND: now also C6.2, P1.10 (P10), P1.13 (P13), P1.19 (P19), P1.26 (P26), P1.29 (P29), P1.33 (P33), P1.40 (P40), P1.5 (P5); no longer C6.1, P1.14 (P14), P1.20 (P20), P1.25 (P25), P1.30 (P30), P1.34 (P34), P1.39 (P39), P1.6 (P6), P1.9 (P9)
- net GPIO04: now also P1.8 (P8); no longer P1.7 (P7)
- net GPIO05: now also P1.30 (P30); no longer P1.29 (P29)
- net GPIO06: now also P1.32 (P32); no longer P1.31 (P31)
- net GPIO12: now also P1.31 (P31); no longer P1.32 (P32)
- net GPIO13: now also P1.34 (P34); no longer P1.33 (P33)
- net GPIO16: now also P1.35 (P35); no longer P1.36 (P36)
- net GPIO17: now also P1.12 (P12); no longer P1.11 (P11)
- net GPIO18: now also P1.11 (P11); no longer P1.12 (P12)
- net GPIO19: now also P1.36 (P36); no longer P1.35 (P35)
- net GPIO20: now also P1.37 (P37); no longer P1.38 (P38)
- net GPIO21: now also P1.39 (P39); no longer P1.40 (P40)
- net GPIO22: now also P1.16 (P16); no longer P1.15 (P15)
- net GPIO23: now also P1.15 (P15); no longer P1.16 (P16)
- net GPIO24: now also P1.17 (P17); no longer P1.18 (P18)
- net GPIO25: now also P1.21 (P21); no longer P1.22 (P22)
- net GPIO26: now also P1.38 (P38); no longer P1.37 (P37)
- net GPIO27: now also P1.14 (P14); no longer P1.13 (P13)
- net ID_SC: now also P1.27 (P27); no longer P1.28 (P28)
- net ID_SD: now also P1.28 (P28); no longer P1.27 (P27)
- net RXD0_GPIO15: now also P1.9 (P9); no longer P1.10 (P10)
- net SCL1_GPIO03: now also P1.6 (P6), J1.1, J2.1, R2.1, R5.1; no longer P1.5 (P5)
- net SDA1_GPIO02: now also P1.4 (P4), J1.2, J2.2, R1.1, R6.1; no longer P1.3 (P3)
- net SPI_CE0_GPIO08: now also P1.23 (P23); no longer P1.24 (P24)
- net SPI_CE1_GPIO07: now also P1.25 (P25); no longer P1.26 (P26)
- net SPI_CLK_GPIO11: now also P1.24 (P24); no longer P1.23 (P23)
- net SPI_MISO_GPIO09: now also P1.22 (P22); no longer P1.21 (P21)
- net SPI_MOSI_GPIO10: now also P1.20 (P20); no longer P1.19 (P19)
- net TXD0_GPIO14: now also P1.7 (P7); no longer P1.8 (P8)
- net at FB3.1: now also P3.1 (P1)
- net at FB4.1: now also P3.2 (P2)
- net at C2.2, C3.1, U2.4 (AIN0): now also R3.2, R4.1
- net at C3.2, C4.1, U2.5 (AIN1): now also J3.4, R3.1
- net at C8.2, C9.1, U2.6 (AIN2): now also J3.2, R7.1
- net at C7.2, C8.1, U2.7 (AIN3): now also R7.2, R8.1
- new net: J3.1, R8.2
- new net: J3.3, R4.2
- new net: J1.3, J2.3
- new net: J1.4, J2.4
- no-connect marks 28 -> 24
Other:
- note added: "Voltage divider: 130:30 = 4 1/3 : 1\n(converting 12V range to 3V3 range)"
- note removed: "0.1% resistors"
- note removed: "Grove connector or bare holes"
- note removed: "Voltage divider: 133:33 = 4 1/33 : 1\n(converting 12V range to 3V3 range)"
