File: octelehat.kicad_pcb (KiCad board)
At the start: 2 copper layers, 65 x 56 mm, 38 parts, among them P1 CONN_02X20, P2 CONN_01X04, P3 CONN_01X04, P4 CONN_01X02, P5 CONN_01X04, P6 CONN_01X04, P7 CONN_01X02, U1 MAX31855, U2 MAX31855, U3 ADS1015

Commit message: PCB work in progress
Parts:
- removed P4, P7: CONN_01X02, hat-parts:Thermocouple
- removed P5, P6: CONN_01X04, Pin_Headers:Pin_Header_Straight_1x04_Pitch2.54mm
- added J1: GROVE-CONNECTOR-DIP-90D_4P-2.0_, SeeedOPL-Connector-2016:HW4-2.0-90D, F.Cu at (72.4, 119.4)
- added J2: GROVE-CONNECTOR-DIP-90D_4P-2.0_, SeeedOPL-Connector-2016:HW4-2.0-90D, F.Cu at (79.0, 145.0)
- added J3: GROVE-CONNECTOR-DIP-90D_4P-2.0_, SeeedOPL-Connector-2016:HW4-2.0-90D, F.Cu at (62.5, 139.2)
- C1, C10, C11, C2, C3, C4, C5, C6, C7, C8, C9: footprint Capacitors_SMD:C_0805_HandSoldering -> Capacitors_SMD:C_0402
- P1: footprint Pin_Headers:Pin_Header_Straight_2x20_Pitch2.54mm -> Socket_Strips:Socket_Strip_Straight_2x20_Pitch2.54mm
- P2, P3: value CONN_01X04 -> CONN_01X02; footprint Pin_Headers:Pin_Header_Straight_1x04_Pitch2.54mm -> hat-parts:Thermocouple
- R1, R2, R5, R6: value 10k -> SMD-RES-10K-1%-1_10W_0603_; footprint Resistors_SMD:R_0805_HandSoldering -> SeeedOPL-Resistor-2016:R0603
- R3, R7: value 100k -> SMD-RES-100K-1%-1_10W_0603_; footprint Resistors_SMD:R_0805_HandSoldering -> SeeedOPL-Resistor-2016:R0603
- R4, R8: value 33k -> SMD-RES-30K-1%-1_10W_0603_; footprint Resistors_SMD:R_0805_HandSoldering -> SeeedOPL-Resistor-2016:R0603
- U1: value MAX31855 -> MAX31855KASA
- U2: value MAX31855 -> ADS1015; footprint hat-parts:SO-8 -> Housings_SSOP:TSSOP-10_3x3mm_Pitch0.5mm
- U3: value ADS1015 -> MAX31855KASA; footprint Housings_SSOP:TSSOP-10_3x3mm_Pitch0.5mm -> hat-parts:SO-8
- moved R4 170.6 mm to (278.3, 122.8)
- moved R3 162.2 mm to (270.0, 123.1)
- moved C2 157.8 mm to (273.7, 133.2)
- moved C6 148.5 mm to (269.5, 133.8), turned to 0 degrees
- moved R5 147.5 mm to (274.2, 122.8), turned to 0 degrees
- moved R8 141.2 mm to (248.7, 149.8)
- moved C4 140.1 mm to (256.1, 143.3)
- moved R1 138.9 mm to (252.9, 132.9), turned to 0 degrees
- moved C7 137.4 mm to (252.4, 143.3)
- moved C3 136.4 mm to (252.4, 147.9)
- moved R2 134.3 mm to (248.7, 132.9)
- moved C9 127.7 mm to (243.9, 130.9)
- moved C1 123.4 mm to (256.1, 147.9), turned to 0 degrees
- moved U3 121.7 mm to (241.0, 149.9), turned to 0 degrees
- moved R7 120.4 mm to (227.5, 150.9)
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Connections:
- C6 pad 1: GND -> +3V3
- C6 pad 2: +3V3 -> GND
- P1 pad 1: /5V -> +3V3
- P1 pad 10: GND -> /RXD0_GPIO15
- P1 pad 11: /GPIO18 -> /GPIO17
- P1 pad 12: /GPIO17 -> /GPIO18
- P1 pad 13: GND -> /GPIO27
- P1 pad 14: /GPIO27 -> GND
- P1 pad 15: /GPIO23 -> /GPIO22
- P1 pad 16: /GPIO22 -> /GPIO23
- P1 pad 17: /GPIO24 -> +3V3
- P1 pad 18: +3V3 -> /GPIO24
- P1 pad 19: GND -> /SPI_MOSI_GPIO10
- P1 pad 2: +3V3 -> /5V
- P1 pad 20: /SPI_MOSI_GPIO10 -> GND
- P1 pad 21: /GPIO25 -> /SPI_MISO_GPIO09
- P1 pad 22: /SPI_MISO_GPIO09 -> /GPIO25
- P1 pad 23: /SPI_CE0_GPIO08 -> /SPI_CLK_GPIO11
- P1 pad 24: /SPI_CLK_GPIO11 -> /SPI_CE0_GPIO08
- P1 pad 25: /SPI_CE1_GPIO07 -> GND
- P1 pad 26: GND -> /SPI_CE1_GPIO07
- P1 pad 27: /ID_SC -> /ID_SD
- P1 pad 28: /ID_SD -> /ID_SC
- P1 pad 29: GND -> /GPIO05
- P1 pad 3: Net-(P1-Pad3) -> /SDA1_GPIO02
- P1 pad 30: /GPIO05 -> GND
- P1 pad 31: /GPIO12 -> /GPIO06
- P1 pad 32: /GPIO06 -> /GPIO12
- P1 pad 33: GND -> /GPIO13
- P1 pad 34: /GPIO13 -> GND
- P1 pad 35: /GPIO16 -> /GPIO19
- P1 pad 36: /GPIO19 -> /GPIO16
- P1 pad 37: /GPIO20 -> /GPIO26
- P1 pad 38: /GPIO26 -> /GPIO20
- P1 pad 39: /GPIO21 -> GND
- P1 pad 4: /SDA1_GPIO02 -> Net-(P1-Pad4)
- P1 pad 40: GND -> /GPIO21
- P1 pad 5: GND -> /SCL1_GPIO03
- P1 pad 6: /SCL1_GPIO03 -> GND
- P1 pad 7: /TXD0_GPIO14 -> /GPIO04
- P1 pad 8: /GPIO04 -> /TXD0_GPIO14
- P1 pad 9: /RXD0_GPIO15 -> GND
- P2 pad 1: /SCL1_GPIO03 -> Net-(FB1-Pad1)
- P2 pad 2: /SDA1_GPIO02 -> Net-(FB2-Pad1)
- P3 pad 1: /SCL1_GPIO03 -> Net-(FB3-Pad1)
- P3 pad 2: /SDA1_GPIO02 -> Net-(FB4-Pad1)
- R1 pad 1: +3V3 -> /SDA1_GPIO02
- R1 pad 2: /SDA1_GPIO02 -> +3V3
- R2 pad 1: +3V3 -> /SCL1_GPIO03
- R2 pad 2: /SCL1_GPIO03 -> +3V3
- R3 pad 1: Net-(C2-Pad2) -> Net-(C3-Pad2)
- R3 pad 2: Net-(C3-Pad2) -> Net-(C2-Pad2)
- R4 pad 1: Net-(P5-Pad1) -> Net-(C2-Pad2)
- R4 pad 2: Net-(C2-Pad2) -> Net-(J3-Pad3)
- R5 pad 1: +3V3 -> /SCL1_GPIO03
- R5 pad 2: /SCL1_GPIO03 -> +3V3
- R6 pad 1: +3V3 -> /SDA1_GPIO02
- R6 pad 2: /SDA1_GPIO02 -> +3V3
- R7 pad 1: Net-(C7-Pad2) -> Net-(C8-Pad2)
- R7 pad 2: Net-(C8-Pad2) -> Net-(C7-Pad2)
- R8 pad 1: Net-(P6-Pad1) -> Net-(C7-Pad2)
- R8 pad 2: Net-(C7-Pad2) -> Net-(J3-Pad1)
- U2 pad 2: Net-(C11-Pad2) -> GND
- U2 pad 3: Net-(C11-Pad1) -> GND
- U2 pad 4: +3V3 -> Net-(C2-Pad2)
- U2 pad 5: /SPI_CLK_GPIO11 -> Net-(C3-Pad2)
- U2 pad 6: /SPI_CE1_GPIO07 -> Net-(C8-Pad2)
- U2 pad 7: /SPI_MISO_GPIO09 -> Net-(C7-Pad2)
- U2 pad 8: (no net) -> +3V3
- U3 pad 2: GND -> Net-(C11-Pad2)
- U3 pad 3: GND -> Net-(C11-Pad1)
- U3 pad 4: Net-(C2-Pad2) -> +3V3
- U3 pad 5: Net-(C3-Pad2) -> /SPI_CLK_GPIO11
- U3 pad 6: Net-(C8-Pad2) -> /SPI_CE1_GPIO07
- U3 pad 7: Net-(C7-Pad2) -> /SPI_MISO_GPIO09
- U3 pad 8: +3V3 -> (no net)

Commit message: adjust design rules
Other:
- net class Default: clearance 0.2 -> 0.25; via_drill 0.4 -> 0.3
- rule trace_clearance: 0.2 -> 0.25
Changed lines of the file:
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@@
   (setup
     (last_trace_width 0.25)
-    (trace_clearance 0.2)
+    (trace_clearance 0.25)
     (zone_clearance 0.508)
     (zone_45_only no)
@@
     (edge_width 0.15)
     (via_size 0.6)
-    (via_drill 0.4)
+    (via_drill 0.3)
     (via_min_size 0.4)
     (via_min_drill 0.3)
@@
   (net 48 "Net-(P1-Pad4)")
   (net_class Default "This is the default net class."
-    (clearance 0.2)
+    (clearance 0.25)
     (trace_width 0.25)
     (via_dia 0.6)
-    (via_drill 0.4)
+    (via_drill 0.3)
     (uvia_dia 0.3)
     (uvia_drill 0.1)

Commit message: work in progress
Parts:
- moved C2 188.8 mm to (85.2, 145.8)
- moved R4 171.1 mm to (109.8, 151.8)
- moved C7 168.0 mm to (85.8, 164.2)
- moved R3 165.8 mm to (108.2, 159.8)
- moved C3 163.7 mm to (88.8, 147.8)
- moved C4 163.4 mm to (92.8, 147.2)
- moved C9 161.5 mm to (84.8, 158.0)
- moved R5 149.0 mm to (125.2, 126.8)
- moved C6 147.2 mm to (122.2, 132.0)
- moved R1 140.8 mm to (113.0, 117.0), turned to 90 degrees
- moved R2 136.4 mm to (113.0, 119.0), turned to 90 degrees
- moved C8 133.0 mm to (88.8, 159.8)
- moved R8 132.0 mm to (116.8, 151.0)
- moved C1 122.6 mm to (135.5, 125.8), turned to 180 degrees
- moved R7 114.0 mm to (113.5, 147.9)
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Connections:
- J1 pad 3: Net-(J1-Pad3) -> +3V3
- J1 pad 4: Net-(J1-Pad4) -> GND
- J2 pad 3: Net-(J1-Pad3) -> +3V3
- J2 pad 4: Net-(J1-Pad4) -> GND
Routing:
- net Net-(FB2-Pad1): track 0.00 -> 6.18 mm
- net Net-(FB4-Pad1): track 0.00 -> 6.06 mm
- net Net-(FB1-Pad1): track 0.00 -> 6.04 mm
- net Net-(FB3-Pad1): track 0.00 -> 5.77 mm
- net Net-(C11-Pad1): track 0.00 -> 5.58 mm
- net Net-(C5-Pad2): track 0.00 -> 5.37 mm
- net Net-(C5-Pad1): track 0.00 -> 5.37 mm
- net Net-(C11-Pad2): track 0.00 -> 5.37 mm
- added copper zone on B.Cu, net GND
Other:
- net class Power added: clearance 0.25, trace_width 0.35, via_dia 0.6, via_drill 0.3
- board text removed: "Voltage 1"
- board text removed: "Voltage 2"

Commit message: rev1 routing
Parts:
- moved C7 51.9 mm to (116.8, 122.7), turned to 90 degrees
- moved C9 51.3 mm to (116.8, 117.9), turned to 90 degrees
- moved C8 48.5 mm to (116.8, 120.2), turned to 90 degrees
- moved R3 47.6 mm to (113.9, 112.5), turned to 90 degrees
- moved C3 44.7 mm to (116.8, 113.0), turned to 90 degrees
- moved C2 43.9 mm to (116.8, 115.3), turned to 90 degrees
- moved C4 43.8 mm to (116.9, 110.7), turned to 90 degrees
- moved R4 37.3 mm to (113.9, 114.7), turned to 270 degrees
- moved R8 30.0 mm to (114.1, 121.2), turned to 270 degrees
- moved R7 29.1 mm to (114.1, 118.8), turned to 270 degrees
- moved J1 24.0 mm to (109.5, 140.0)
- moved J3 24.0 mm to (109.5, 116.0)
- moved R2 18.1 mm to (115.6, 137.0)
- moved R1 18.1 mm to (115.6, 134.9)
- moved U2 16.3 mm to (121.9, 115.6), turned to 270 degrees
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Connections:
- J3 pad 2: Net-(C8-Pad2) -> Net-(C7-Pad2)
- R8 pad 1: Net-(C7-Pad2) -> Net-(C8-Pad2)
Routing:
- net GND: track 0.00 -> 368.8 mm, vias 0 -> 9
- net +3V3: track 0.00 -> 142.1 mm, vias 0 -> 2
- net /SCL1_GPIO03: track 0.00 -> 69.6 mm, vias 0 -> 2
- net /SDA1_GPIO02: track 0.00 -> 59.2 mm, vias 0 -> 4
- net /SPI_MISO_GPIO09: track 0.00 -> 41.0 mm, vias 0 -> 2
- net /SPI_CLK_GPIO11: track 0.00 -> 36.4 mm, vias 0 -> 2
- net /SPI_CE1_GPIO07: track 0.00 -> 23.0 mm
- net /SPI_CE0_GPIO08: track 0.00 -> 20.6 mm
- net Net-(C7-Pad2): track 0.00 -> 17.0 mm, vias 0 -> 2
- net Net-(C3-Pad2): track 0.00 -> 14.4 mm
- net Net-(C2-Pad2): track 0.00 -> 12.0 mm
- net Net-(C8-Pad2): track 0.00 -> 10.1 mm
- net Net-(J3-Pad1): track 0.00 -> 4.70 mm
- net Net-(J3-Pad3): track 0.00 -> 3.78 mm
- net Net-(FB3-Pad1): track 5.77 -> 7.92 mm
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- added copper zone on F.Cu, net GND
Other:
- net class Default: clearance 0.25 -> 0.2; via_dia 0.6 -> 0.5
- net class Power: clearance 0.25 -> 0.2; trace_width 0.35 -> 0.3; via_dia 0.6 -> 0.5
- rule trace_clearance: 0.25 -> 0.2
- board text added: "+"
- board text added: "-"
- board text added: "100K+30K 130:30 divider"
- board text added: "2017 rev1 CERN OHL 1.2"
- board text added: "ADS1015"
- board text added: "GND"
- board text added: "SCL"
- board text added: "SDA"
- board text added: "V1"
- board text added: "V2"
- board text added: "VCC"
- board text added: "Voltage"
- board text removed: "2017 rev0 CERN OHL 1.2"

Commit message: revised
Routing:
- net +3V3: track 142.1 -> 119.6 mm, vias 2 -> 0
- net GND: track 368.8 -> 374.1 mm
Other:
- board text added: "EPEAK Gear - TeVo X2"
- board text removed: "Overclocking Telemetry HAT"

Commit message: design update
Parts:
- FB1, FB2, FB3, FB4: footprint Resistors_SMD:R_0603_HandSoldering -> SeeedOPL-Inductor-2016:L0603
- moved C7 12.0 mm to (117.5, 110.7), turned to 180 degrees
- moved R6 10.5 mm to (122.5, 109.5), turned to 180 degrees
- moved R5 8.80 mm to (120.3, 109.5), turned to 180 degrees
- moved C6 8.41 mm to (123.5, 112.0), turned to 0 degrees
- moved C8 7.58 mm to (117.5, 112.7), turned to 180 degrees
- moved R8 7.40 mm to (114.1, 113.8)
- moved R7 7.24 mm to (114.1, 111.6)
- moved C4 6.18 mm to (117.4, 116.8), turned to 0 degrees
- moved C3 5.99 mm to (117.4, 119.0), turned to 180 degrees
- moved R4 5.88 mm to (114.1, 120.5)
- moved C2 5.72 mm to (117.4, 121.0), turned to 180 degrees
- moved R3 5.67 mm to (114.1, 118.1)
- moved C9 3.12 mm to (117.5, 114.8), turned to 0 degrees
- moved U2 0.28 mm to (121.9, 115.9), turned to 90 degrees
Connections:
- J3 pad 2: Net-(C7-Pad2) -> Net-(C3-Pad2)
- J3 pad 4: Net-(C3-Pad2) -> Net-(C7-Pad2)
- R4 pad 2: Net-(J3-Pad3) -> Net-(J3-Pad1)
- R8 pad 2: Net-(J3-Pad1) -> Net-(J3-Pad3)
Routing:
- net GND: track 374.1 -> 415.4 mm, vias 9 -> 13
- net /SCL1_GPIO03: track 69.6 -> 56.0 mm
- net Net-(C3-Pad2): track 14.4 -> 20.0 mm
- net Net-(C8-Pad2): track 10.1 -> 14.9 mm
- net +3V3: track 119.6 -> 123.2 mm
- net /SDA1_GPIO02: track 59.2 -> 61.5 mm, vias 4 -> 3
- net Net-(C2-Pad2): track 12.0 -> 13.6 mm
- net Net-(J3-Pad3): track 3.78 -> 4.37 mm
- net Net-(C7-Pad2): track 17.0 -> 17.2 mm, vias 2 -> 0
Other:
- board text added: "100K+30K 130:30 divider to 3V3"
- board text added: "EPEAK Gear TeVo X2"
- board text removed: "100K+30K 130:30 divider"
- board text removed: "EPEAK Gear - TeVo X2"

Commit message: update voltage divider part of circuit
Other:
- board text added: "2017 rev2 CERN OHL 1.2"
- board text removed: "2017 rev1 CERN OHL 1.2"
Changed lines of the file:
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@@
   (title_block
     (title "Overclocking Telemetry HAT for Raspberry Pi 3")
-    (date 2017-04-10)
-    (rev 1)
+    (date 2017-05-19)
+    (rev 2)
     (company Moonpunch.org)
     (comment 1 "CERN OHL 1.2")
@@
     (effects (font (size 1 1) (thickness 0.25)))
   )
-  (gr_text "2017 rev1\nCERN OHL 1.2" (at 160.925 148.975 90) (layer F.SilkS)
+  (gr_text "2017 rev2\nCERN OHL 1.2" (at 160.925 148.975 90) (layer F.SilkS)
     (effects (font (size 1.2 1.2) (thickness 0.3)) (justify left))
   )
@@
   (gr_arc (start 162 103) (end 162 100) (angle 90) (layer Edge.Cuts) (width 0.15))
   (gr_line (start 103 100) (end 162 100) (angle 90) (layer Edge.Cuts) (width 0.15))
-  (segment (start 116.342 134.88) (end 116.342 134.158) (width 0.3) (layer F.Cu) (net 1) (status 400000))
+  (segment (start 116.342 134.88) (end 116.342 134.158) (width 0.3) (layer F.Cu) (net 1))
   (segment (start 125.66 124.84) (end 125.66 121.3) (width 0.3) (layer F.Cu) (net 1))
   (segment (start 116.342 134.158) (end 125.66 124.84) (width 0.3) (layer F.Cu) (net 1))
-  (segment (start 122.95 112) (end 122.95 112.08) (width 0.3) (layer F.Cu) (net 1) (status C00000))
-  (segment (start 122.95 112.08) (end 125.66 114.79) (width 0.3) (layer F.Cu) (net 1) (status 400000))
+  (segment (start 122.95 112) (end 122.95 112.08) (width 0.3) (layer F.Cu) (net 1))
+  (segment (start 122.95 112.08) (end 125.66 114.79) (width 0.3) (layer F.Cu) (net 1))
   (segment (start 125.66 114.79) (end 125.66 121.3) (width 0.3) (layer F.Cu) (net 1))
   (segment (start 128.28 123.92) (end 133.66 123.92) (width 0.3) (layer F.Cu) (net 1))

Commit message: updated rev2
Changed lines of the file:
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@@
     (effects (font (size 1.5 1.5) (thickness 0.3)))
   )
-  (gr_text V2 (at 111.2 109.89) (layer F.SilkS)
+  (gr_text V2 (at 110.236 109.982) (layer F.SilkS)
     (effects (font (size 1 1) (thickness 0.25)))
   )
-  (gr_text V1 (at 111.17 121.99) (layer F.SilkS)
+  (gr_text V1 (at 110.236 122.174) (layer F.SilkS)
     (effects (font (size 1 1) (thickness 0.25)))
   )
